File: LED-DriverPCB/LED-DriverPCB.kicad_sch (KiCad schematic)
At the start: 51 parts, among them J1 Screw_Terminal_01x03, J12 Screw_Terminal_01x02, J13 Screw_Terminal_01x02, J14 Screw_Terminal_01x02, J15 Screw_Terminal_01x02, J16 Screw_Terminal_01x02, J17 Screw_Terminal_01x02, J18 Screw_Terminal_01x02, J19 Screw_Terminal_01x02, J2 Screw_Terminal_01x03, J20 Conn_ARM_SWD_TagConnect_TC2030, J3 Screw_Terminal_01x03, J4 Screw_Terminal_01x03, J5 Screw_Terminal_01x03, J6 Screw_Terminal_01x03, J7 Screw_Terminal_01x03, J8 Screw_Terminal_01x03, J9 USB_C_Receptacle_USB2.0_16P, U1 STM32F103RCTx, U2 TXB0108PW, U3 AMS1117-3.3, U4 USBLC6-2SC6, X1 8MHz

Commit message: Finalized layout
Parts:
- C1, C2: value C -> 10p; JLCPCB Part # (none) -> C161145
- C10, C13, C14, C3, C4, C5, C6, C7, C8: JLCPCB Part # (none) -> C1590
- C11, C15, C9: JLCPCB Part # (none) -> C15850
- C12: JLCPCB Part # (none) -> C45783
- J9: JLCPCB Part # (none) -> C165948
- R1: JLCPCB Part # (none) -> C5184132
- R2, R3: JLCPCB Part # (none) -> C23186
- R4: JLCPCB Part # (none) -> C861451
- R5: JLCPCB Part # (none) -> C22843
- U1: JLCPCB Part # (none) -> C8323
- U2: JLCPCB Part # (none) -> C53406
- U3: JLCPCB Part # (none) -> C6186
- U4: JLCPCB Part # (none) -> USBLC6-2SC6
- X1: JLCPCB Part # (none) -> C400090
